File: Hardware/PCB.brd (EAGLE design)
At the start: 170.2 x 111.2 mm, 103 parts, among them IC1 BD5229G-TR, IC4 XC6220A331MR-G, J1 FH34SRJ-24S-0.5SH_99_, J2 SAMACSYS_PARTS_USB4110-GF-A, J3 QWIIC_RIGHT_ANGLE, J4 112A-TAAR-R03_ATTEND, Q1 20V/4.2A/52mΩ/1.4W, Q2 SI1308EDL-T1-GE3, Q3 20V/4.2A/52mΩ/1.4W, U1 W25Q512JVEIQ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

Commit message: Final version
Updated files to solve #1 #2 #3 #4 #5.
Routing:
- net GND: vias 12 -> 32
Changed lines of the file:
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@@
 <layer number="16" name="Bottom" color="1" fill="1" visible="no" active="yes"/>
 <layer number="17" name="Pads" color="2" fill="1" visible="no" active="yes"/>
-<layer number="18" name="Vias" color="2" fill="1" visible="no" active="yes"/>
+<layer number="18" name="Vias" color="2" fill="1" visible="yes" active="yes"/>
 <layer number="19" name="Unrouted" color="6" fill="1" visible="no" active="yes"/>
 <layer number="20" name="Dimension" color="24" fill="1" visible="no" active="yes"/>
@@
 <layer number="33" name="tFinish" color="6" fill="3" visible="no" active="yes"/>
 <layer number="34" name="bFinish" color="6" fill="6" visible="no" active="yes"/>
-<layer number="35" name="tGlue" color="7" fill="4" visible="no" active="yes"/>
+<layer number="35" name="tGlue" color="7" fill="4" visible="yes" active="yes"/>
 <layer number="36" name="bGlue" color="7" fill="5" visible="no" active="yes"/>
-<layer number="37" name="tTest" color="7" fill="1" visible="no" active="yes"/>
+<layer number="37" name="tTest" color="7" fill="1" visible="yes" active="yes"/>
 <layer number="38" name="bTest" color="7" fill="1" visible="no" active="yes"/>
 <layer number="39" name="tKeepout" color="4" fill="11" visible="no" active="yes"/>
@@
 <via x="62.595" y="105.36" extent="1-16" drill="0.35" alwaysstop="yes">
 </via>
+<via x="66.385" y="48.725" extent="1-16" drill="0.35" alwaysstop="yes">
+</via>
+<via x="28.825" y="56.335" extent="1-16" drill="0.35" alwaysstop="yes">
+</via>
+<via x="21.335" y="72.8" extent="1-16" drill="0.35" alwaysstop="yes">
+</via>
+<via x="24.525" y="38.275" extent="1-16" drill="0.35" alwaysstop="yes">
+</via>
+<via x="56.25" y="107.31" extent="1-16" drill="0.35" alwaysstop="yes">
+</via>
+<via x="56.25" y="103.055" extent="1-16" drill="0.35" alwaysstop="yes">
+</via>
+<via x="28.68" y="64.08" extent="1-16" drill="0.35" alwaysstop="yes">
+</via>
+<via x="30.02" y="60.375" extent="1-16" drill="0.35" alwaysstop="yes">
+</via>
+<via x="30.045" y="41.725" extent="1-16" drill="0.35" alwaysstop="yes">
+</via>
+<via x="90.525" y="49.07" extent="1-16" drill="0.35" alwaysstop="yes">
+</via>
+<via x="105.38" y="48.66" extent="1-16" drill="0.35" alwaysstop="yes">
+</via>
+<via x="61.83" y="43.99" extent="1-16" drill="0.35" alwaysstop="yes">
+</via>
+<via x="29.585" y="45.22" extent="1-16" drill="0.35" alwaysstop="yes">
+</via>
+<via x="17.1" y="48.595" extent="1-16" drill="0.35" alwaysstop="yes">
+</via>
+<via x="151.895" y="32.485" extent="1-16" drill="0.35" alwaysstop="yes">
+</via>
+<via x="35.07" y="56.48" extent="1-16" drill="0.35" alwaysstop="yes">
+</via>
+<via x="29.64" y="51.52" extent="1-16" drill="0.35" alwaysstop="yes">
+</via>
+<via x="10.97" y="80.465" extent="1-16" drill="0.35" alwaysstop="yes">
+</via>
+<via x="10.08" y="96.745" extent="1-16" drill="0.35" alwaysstop="yes">
+</via>
+<via x="33.25" y="36.865" extent="1-16" drill="0.35" alwaysstop="yes">
+</via>
 </signal>
 <signal name="VUSB" class="1">
@@
 <mfgpreviewcolor name="silkscreencolor" color="0xFFFEFEFE"/>
 <mfgpreviewcolor name="backgroundcolor" color="0xFF282828"/>
-<mfgpreviewcolor name="coppercolor" color="0xCCC90C0C"/>
+<mfgpreviewcolor name="coppercolor" color="0xCCFFBB00"/>
 <mfgpreviewcolor name="substratecolor" color="0xFF786E46"/>
 </mfgpreviewcolors>
